File: OpenRadiosondePCB/OpenRadiosondePCB.kicad_sch (KiCad schematic)
At the start: 72 parts, among them IC1 SI4468-A2A-IMR, IC2 IS66WVS1M8BLL-104NLI, J1 ICSP, J2 GPS_ANT, J3 RF_OUT_70CM, J4 RF_OUT_2M, J5 SPI3, J6 CAM, U1 STM32L476RGTx, U2 AS179-92LF, U3 MAX-M10S, U4 LPS22HB, U5 TPS61201DRC, U6 UART_DEBUG, Y2 FT2MNTUM-30.0-T1

Commit message: Finalizing schematic, some more pin changes
Parts:
- removed C8: 1uF, Capacitor_SMD:C_0402_1005Metric, symbol Device:C
- removed C9: 10uF, Capacitor_SMD:C_0402_1005Metric, symbol Device:C
- removed J5: SPI3, symbol CustomLibs:SPI3
- removed L1: 100nH, Inductor_SMD:L_0402_1005Metric, symbol Device:L
- added C24: 1uF, Capacitor_SMD:C_0402_1005Metric, symbol Device:C
- added C25: 10uF, Capacitor_SMD:C_0402_1005Metric, symbol Device:C
- added J5: EXPANSION, Connector_PinHeader_2.54mm:PinHeader_1x08_P2.54mm_Vertical, symbol CustomLibs:EXPANSION
- added J7: Micro_SD_Card, CustomLibs:1140084168, symbol Connector:Micro_SD_Card
- added J8: PWR_IN, Connector_PinHeader_2.54mm:PinHeader_1x02_P2.54mm_Vertical, symbol CustomLibs:PWR_IN
- added L11: 100nH, Inductor_SMD:L_0402_1005Metric, symbol Device:L
- added NT1, NT2, NT3: NetTie_2, symbol Device:NetTie_2
- added R23: 4.7k, Resistor_SMD:R_0402_1005Metric, symbol Device:R
- IC2: footprint SOIC127P600X175-8N -> CustomLibs:SOIC127P600X175-8N
- J1: footprint (none) -> Connector_PinHeader_2.54mm:PinHeader_1x05_P2.54mm_Vertical
- J6: footprint (none) -> CustomLibs:LPS3015
- L2: footprint Inductor_SMD:L_0402_1005Metric -> Inductor_SMD:L_Coilcraft_LPS3010
- R16, R17, R20: value 1k -> 4.7k; footprint (none) -> Resistor_SMD:R_0402_1005Metric
- R18: footprint (none) -> Resistor_SMD:R_0402_1005Metric
- R19: value 220R -> 4.7k; footprint (none) -> Resistor_SMD:R_0402_1005Metric
- R21, R22: value 220R -> 1k; footprint (none) -> Resistor_SMD:R_0402_1005Metric
- R5: value 150k -> 180k
Connections:
- net SPI3_MISO is gone; now on net CAM_HREF: U1.52 (PC11)
- net SPI3_OUT_CS is gone; now on net +3V3: R20.1
- net SPI3_OUT_MISO is gone; now on net DEBUG_RX: R21.1
- net SPI3_OUT_MOSI is gone; now on net +3V3: R19.1
- net SPI3_OUT_SCK is gone; now on net DEBUG_TX: R22.1
- net SPI3_SCK is gone; now on net CAM_PCLK: U1.51 (PC10)
- net +3V3: now also R16.1, R17.2, J5.1 (3.3V), J7.4 (VDD), L11.2, R23.1
- net +BATT: now also J8.1 (BAT)
- net CAM_D0: now also U1.26 (PB0)
- net CAM_D1: now also U1.27 (PB1)
- net CAM_D2: now also U1.28 (PB2)
- net CAM_D3: now also U1.24 (PC4)
- net CAM_D4: now also U1.25 (PC5)
- net CAM_D5: now also U1.36 (PB15)
- net CAM_D6: now also U1.37 (PC6)
- net CAM_D7: now also U1.38 (PC7)
- net CAM_PDN: now also R19.2, U1.35 (PB14)
- net CAM_RST: now also U1.33 (PB12)
- net CAM_VS: now also U1.40 (PC9)
- net CAM_XCLK: now also U1.41 (PA8)
- net DEBUG_RX: no longer U6.3 (RX)
- net DEBUG_TX: no longer U6.2 (TX)
- net GND: now also C24.2, C25.2, J5.5 (GND), J7.6 (VSS), J7.9 (SHIELD), J8.2 (GND)
- net GPS_PPS: now also U1.56 (PB4)
- net GPS_RESET: now also U1.57 (PB5)
- net LED_B: now also U1.4 (PC15)
- net LED_G: now also U1.3 (PC14)
- net LED_R: now also U1.2 (PC13)
- net LPS22_CS: now also R20.2, U1.17 (PA3)
- net LPS22_MISO: now also NT2.2; no longer IC2.2 (SO/SIO1), U1.10 (PC2)
- net LPS22_MOSI: now also NT3.2; no longer IC2.5 (SI/SIO0)
- net LPS22_SCLK: now also NT1.1; no longer IC2.6 (CLK)
- net RADIO_CS: now also R17.1, U1.15 (PA1)
- net RADIO_RAW_MOD: now also U1.50 (PA15)
- net RADIO_SDN: now also U1.16 (PA2)
- net RF_SELECT_2M: now also U1.61 (PB8), U2.6 (V2); no longer R16.2
- net RF_SELECT_70CM: now also U1.62 (PB9), U2.4 (V1); no longer R17.2
- net SRAM_CS: now also R16.2
- net at R21.2: now also U6.3 (RX)
- net at U1.13 (VDDA): now also C24.1, C25.1, L11.1
- net PA4: now reaches U1.20 (PA4)
- net PA4: now also J5.2 (PA4)
- net SD_DAT0: now reaches U1.39 (PC8)
- net SD_DAT0: now also J7.7 (DAT0)
- net PA11: now reaches U1.44 (PA11)
- net PA11: now also J5.3 (PA11)
- net PA12: now reaches U1.45 (PA12)
- net PA12: now also J5.4 (PA12)
- net SD_CMD: now reaches U1.54 (PD2)
- net SD_CMD: now also J7.3 (CMD)
- net SD_CS: now reaches U1.55 (PB3)
- net SD_CS: now also J7.2 (DAT3/CD), R23.2
- net at R22.2: now also U6.2 (TX)
- net SPI3_MOSI renamed SD_CLK
- net SD_CLK: now also J7.5 (CLK)
- new net SRAM_MISO: IC2.2 (SO/SIO1), NT2.1, U1.10 (PC2)
- new net SRAM_MOSI: IC2.5 (SI/SIO0), NT3.1
- new net SRAM_SCLK: IC2.6 (CLK), NT1.2
- no-connect marks 15 -> 20
Other:
- note added: "???"
- note added: "External FET?"
- moved on the sheet: C10, C16, C17, C18, C19, C20, C21, C22, C23, C5, C7, IC1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

Commit message: Working on PCB design
Parts:
- removed J7: Micro_SD_Card, CustomLibs:1140084168, symbol Connector:Micro_SD_Card
- removed NT1, NT2, NT3: NetTie_2, symbol Device:NetTie_2
- removed R18: 180k, Resistor_SMD:R_0402_1005Metric, symbol Device:R
- added C26, C9: 100nF, Capacitor_SMD:C_0603_1608Metric, symbol Device:C
- added C27: 100pF, Capacitor_SMD:C_0603_1608Metric, symbol Device:C
- added C8: 2.2uF, Capacitor_SMD:C_0603_1608Metric, symbol Device:C
- added J9: 1140084168, 1140084168, symbol CustomLibs:1140084168
- C1, C10, C11, C12, C13, C14, C15, C16, C17, C18, C19, C2, C20, C21, C22, C23, C24, C25, C3, C5, C6, C7: footprint Capacitor_SMD:C_0402_1005Metric -> Capacitor_SMD:C_0603_1608Metric
- C4: value 1nF -> 100pF; footprint Capacitor_SMD:C_0402_1005Metric -> Capacitor_SMD:C_0603_1608Metric
- J5: footprint Connector_PinHeader_2.54mm:PinHeader_1x08_P2.54mm_Vertical -> Connector_PinHeader_2.54mm:PinHeader_1x04_P2.54mm_Vertical
- J6: footprint CustomLibs:LPS3015 -> Connector_PinHeader_2.54mm:PinHeader_2x09_P2.54mm_Vertical
- L10, L11, L3, L4, L5, L6, L7, L8, L9: footprint Inductor_SMD:L_0402_1005Metric -> Inductor_SMD:L_0603_1608Metric
- L2: footprint Inductor_SMD:L_Coilcraft_LPS3010 -> CustomLibs:LPS3015
- R1, R10, R11, R12, R13, R14, R15, R16, R17, R19, R2, R20, R21, R22, R23, R3, R4, R5, R6, R7, R8, R9: footprint Resistor_SMD:R_0402_1005Metric -> Resistor_SMD:R_0603_1608Metric
Connections:
- net SRAM_MISO is gone; now on net LPS22_MISO: IC2.2 (SO/SIO1), U1.10 (PC2)
- net SRAM_MOSI is gone; now on net LPS22_MOSI: IC2.5 (SI/SIO0)
- net SRAM_SCLK is gone; now on net LPS22_SCLK: IC2.6 (CLK)
- net +3V3: now also C26.1, C27.1, C8.1, C9.1, J9.4 (SUPPLY_VOLTAGE)
- net GND: now also J5.4 (GND), C26.2, C27.2, C8.2, C9.2, J9.10, J9.11, J9.12, J9.6 (SUPPLY_VOLTAGE_GND); no longer J5.5 (GND)
- net SD_CLK: now also J9.5 (CLOCK)
- net SD_CMD: now also J9.3 (COMMAND/RESPONSE)
- net SD_CS: now also J9.2 (CARD_DETECT_/_DATE_LINE_[BIT_3])
- net SD_DAT0: now also J9.7 (DATE_LINE_[BIT_0])
- net SRAM_CS: now also U1.45 (PA12)
- removed net PA12: J5.4 (PA12), U1.45 (PA12)
- now unconnected: S1.MP2, S1.MP3, S1.MP4
- no-connect marks 20 -> 27
Other:
- moved on the sheet: R23
