File: OpenRadiosondePCB/OpenRadiosondePCB.kicad_sch (KiCad schematic)
At the start: 78 parts, among them IC1 SI4468-A2A-IMR, IC2 IS66WVS1M8BLL-104NLI, J1 ICSP, J2 GPS_ANT, J3 RF_OUT_70CM, J4 RF_OUT_2M, J5 EXPANSION, J6 CAM, J8 PWR_IN, J9 1140084168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

Commit message: More PCB work
Parts:
- L4, L5, L6, L7, L8, L9: footprint Inductor_SMD:L_0603_1608Metric -> Inductor_SMD:L_0805_2012Metric
Changed lines of the file:
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@@
 			)
 		)
-		(property "Footprint" "Inductor_SMD:L_0603_1608Metric"
+		(property "Footprint" "Inductor_SMD:L_0805_2012Metric"
 			(at 360.68 86.36 0)
 			(effects
@@
 			)
 		)
-		(property "Footprint" "Inductor_SMD:L_0603_1608Metric"
+		(property "Footprint" "Inductor_SMD:L_0805_2012Metric"
 			(at 347.98 62.23 0)
 			(effects
@@
 			)
 		)
-		(property "Footprint" "Inductor_SMD:L_0603_1608Metric"
+		(property "Footprint" "Inductor_SMD:L_0805_2012Metric"
 			(at 335.28 62.23 0)
 			(effects
@@
 			)
 		)
-		(property "Footprint" "Inductor_SMD:L_0603_1608Metric"
+		(property "Footprint" "Inductor_SMD:L_0805_2012Metric"
 			(at 335.28 86.36 0)
 			(effects
@@
 			)
 		)
-		(property "Footprint" "Inductor_SMD:L_0603_1608Metric"
+		(property "Footprint" "Inductor_SMD:L_0805_2012Metric"
 			(at 360.68 62.23 0)
 			(effects
@@
 			)
 		)
-		(property "Footprint" "Inductor_SMD:L_0603_1608Metric"
+		(property "Footprint" "Inductor_SMD:L_0805_2012Metric"
 			(at 347.98 86.36 0)
 			(effects
