File: OpenRadiosondePCB/OpenRadiosondePCB.kicad_pcb (KiCad board)
At the start: 2 copper layers, 74 parts, among them IC1 SI4468-A2A-IMR, IC2 IS66WVS1M8BLL-104NLI, J1 ICSP, J2 GPS_ANT, J3 RF_OUT_70CM, J4 RF_OUT_2M, J5 EXPANSION, J6 CAM, J7 Micro_SD_Card, U1 STM32L476RGTx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

Commit message: Working on PCB design
Parts:
- removed J7: Micro_SD_Card, CustomLibs:1140084168
- removed L1: 100nH, Inductor_SMD:L_0402_1005Metric
- removed R18: 180k, Resistor_SMD:R_0402_1005Metric
- added C24: 1uF, Capacitor_SMD:C_0603_1608Metric, F.Cu at (119.9, 42.0)
- added C25: 10uF, Capacitor_SMD:C_0603_1608Metric, F.Cu at (119.9, 43.6)
- added C26: 100nF, Capacitor_SMD:C_0603_1608Metric, B.Cu at (108.0, 63.5)
- added C27: 100pF, Capacitor_SMD:C_0603_1608Metric, B.Cu at (108.0, 65.0)
- added J8: PWR_IN, Connector_PinHeader_2.54mm:PinHeader_1x02_P2.54mm_Vertical, F.Cu at (130.5, 34.4)
- added J9: 1140084168, CustomLibs:1140084168, F.Cu at (125.0, 61.0)
- added L11: 100nH, Inductor_SMD:L_0603_1608Metric, F.Cu at (117.6, 41.2)
- C1, C12, C14, C15, C16, C17, C18, C19, C2, C20, C22, C23, C3, C7: footprint Capacitor_SMD:C_0402_1005Metric -> Capacitor_SMD:C_0603_1608Metric
- C10, C11, C13, C21, C5, C6: footprint Capacitor_SMD:C_0402_1005Metric -> Capacitor_SMD:C_0603_1608Metric; moved to B.Cu
- C4: value 1nF -> 100pF; footprint Capacitor_SMD:C_0402_1005Metric -> Capacitor_SMD:C_0603_1608Metric
- C8: value 1uF -> 2.2uF; footprint Capacitor_SMD:C_0402_1005Metric -> Capacitor_SMD:C_0603_1608Metric; moved to B.Cu
- C9: value 10uF -> 100nF; footprint Capacitor_SMD:C_0402_1005Metric -> Capacitor_SMD:C_0603_1608Metric; moved to B.Cu
- IC1, U2, U5: moved to B.Cu
- J5: footprint Connector_PinHeader_2.54mm:PinHeader_1x08_P2.54mm_Vertical -> Connector_PinHeader_2.54mm:PinHeader_1x04_P2.54mm_Vertical
- J6: footprint CustomLibs:LPS3015 -> Connector_PinHeader_2.54mm:PinHeader_2x09_P2.54mm_Vertical
- L10: footprint Inductor_SMD:L_0402_1005Metric -> Inductor_SMD:L_0603_1608Metric; moved to B.Cu
- L2: footprint Inductor_SMD:L_Coilcraft_LPS3010 -> CustomLibs:LPS3015; moved to B.Cu
- L3, L4, L5, L6, L7, L8, L9: footprint Inductor_SMD:L_0402_1005Metric -> Inductor_SMD:L_0603_1608Metric
- R1, R10, R11, R12, R16, R19, R2, R21, R22, R3, R4, R5: footprint Resistor_SMD:R_0402_1005Metric -> Resistor_SMD:R_0603_1608Metric
- R13, R14, R15, R17, R20, R23, R6, R7, R8, R9: footprint Resistor_SMD:R_0402_1005Metric -> Resistor_SMD:R_0603_1608Metric; moved to B.Cu
- moved J3 113.3 mm to (127.7, 75.4), turned to 180 degrees
- moved D2 110.5 mm to (127.0, 49.4), turned to 90 degrees
- moved L2 99.1 mm to (118.6, 34.7), turned to -90 degrees
- moved L6 95.1 mm to (120.5, 75.4)
- moved R5 93.7 mm to (129.9, 38.0)
- moved L5 93.2 mm to (117.5, 75.4)
- moved L4 91.5 mm to (114.5, 75.4)
- moved R4 90.7 mm to (126.9, 38.0), turned to 180 degrees
- moved R16 90.0 mm to (130.3, 46.8)
- moved R1 88.7 mm to (123.4, 47.8)
- moved R2 88.6 mm to (123.4, 49.3)
- moved R3 88.5 mm to (123.4, 50.8)
- moved R8 86.7 mm to (125.8, 31.7)
- moved R15 86.6 mm to (124.1, 26.6), turned to -90 degrees
- moved L10 85.1 mm to (111.6, 68.8)
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Connections:
- C8 pad 1: Net-(U1-VDDA) -> +3V3
- C9 pad 1: Net-(U1-VDDA) -> +3V3
- J5 pad 3: /PC9 -> /PA11
- J5 pad 4: /PA11 -> GND
- S1 pad MP1: Net-(R18-Pad2) -> unconnected-(S1-PadMP1)
- S1 pad MP2: Net-(R18-Pad1) -> unconnected-(S1-PadMP2)
- S1 pad MP3: Net-(R18-Pad1) -> unconnected-(S1-PadMP3)
- S1 pad MP4: Net-(R18-Pad1) -> unconnected-(S1-PadMP4)
- U1 pad 40: /PC9 -> /CAM_VS
- U1 pad 45: /PA10 -> /SRAM_CS
- U1 pad 51: /PC10 -> /CAM_PCLK
- U1 pad 52: /PC11 -> /CAM_HREF
Routing:
- net +3V3: track 0.00 -> 173.7 mm, vias 0 -> 10
- net /PA4: track 0.00 -> 53.6 mm, vias 0 -> 2
- net /CAM_HREF: track 0.00 -> 39.4 mm, vias 0 -> 4
- net /CAM_D7: track 0.00 -> 38.9 mm, vias 0 -> 3
- net /RF_SELECT_2M: track 0.00 -> 37.9 mm, vias 0 -> 4
- net /RADIO_SCK: track 0.00 -> 35.6 mm, vias 0 -> 1
- net /GPS_SCL: track 0.00 -> 35.5 mm, vias 0 -> 3
- net /RF_SELECT_70CM: track 0.00 -> 35.3 mm, vias 0 -> 1
- net /RADIO_MISO: track 0.00 -> 34.9 mm, vias 0 -> 1
- net /RADIO_MOSI: track 0.00 -> 34.6 mm, vias 0 -> 1
- net GND: track 0.00 -> 34.4 mm
- net +BATT: track 0.00 -> 33.2 mm, vias 0 -> 2
- net /CAM_D5: track 0.00 -> 33.0 mm, vias 0 -> 4
- net /SD_CS: track 0.00 -> 30.3 mm, vias 0 -> 1
- net /SRAM_CS: track 0.00 -> 28.7 mm, vias 0 -> 2
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- added copper zone on B.Cu, net GND
- added copper zone on F.Cu, net GND
Other:
- board outline added: 40 x 64.2 mm
- board text added: "11pF"
- board text added: "13pF"
- board text added: "7.5pF"
- board text added: "C16"
- board text added: "C17"
- board text added: "C7"

Commit message: Rounting (almost) all traces again.
Parts:
- C14: moved to B.Cu
- L4, L5, L6, L7, L8, L9: footprint Inductor_SMD:L_0603_1608Metric -> Inductor_SMD:L_0805_2012Metric
- R8, R9: moved to F.Cu
- moved C15 3.40 mm to (108.5, 60.1), turned to -90 degrees
- moved L3 2.66 mm to (108.5, 57.1), turned to -90 degrees
- moved C22 1.40 mm to (124.9, 75.4)
- moved C23 1.15 mm to (100.0, 75.4)
- moved L6 1.12 mm to (121.6, 75.4)
- moved L9 0.88 mm to (103.3, 75.4)
- moved C17 0.81 mm to (119.8, 77.7)
- moved C20 0.57 mm to (105.2, 77.8)
- moved L5 0.57 mm to (118.1, 75.4)
- moved C18 0.38 mm to (111.3, 77.8)
- moved C7 0.34 mm to (113.5, 77.8)
- moved L8 0.32 mm to (106.8, 75.4)
- moved C16 0.28 mm to (116.3, 77.8)
- moved R9 0.24 mm to (123.0, 31.8)
- moved R8 0.21 mm to (126.0, 31.8)
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Routing:
- net /GPS_SDA: track 19.8 -> 55.2 mm, vias 2 -> 5
- net GND: track 34.4 -> 0.00 mm
- net +3V3: track 173.7 -> 207.3 mm, vias 10 -> 9
- net /CAM_PCLK: track 0.00 -> 32.4 mm, vias 0 -> 1
- net /CAM_VS: track 0.00 -> 31.2 mm, vias 0 -> 1
- net /SRAM_CS: track 28.7 -> 2.13 mm, vias 2 -> 0
- net /SD_CS: track 30.3 -> 4.71 mm, vias 1 -> 2
- net /DEBUG_RX: track 24.5 -> 0.00 mm
- net /DEBUG_TX: track 23.9 -> 0.00 mm
- net /NRST: track 2.92 -> 24.2 mm, vias 1 -> 2
- net /SD_CMD: track 22.6 -> 1.66 mm, vias 0 -> 1
- net /GPS_TX: track 0.00 -> 20.4 mm
- net /PA11: track 1.89 -> 21.9 mm, vias 0 -> 3
- net /GPS_RX: track 0.00 -> 19.5 mm
- net /CAM_D5: track 33.0 -> 13.9 mm, vias 4 -> 1
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
Commit message: More PCB work
Routing:
- net /DEBUG_TX: track 0.00 -> 30.6 mm, vias 0 -> 8
- net /DEBUG_RX: track 0.00 -> 29.4 mm, vias 0 -> 2
- net /SRAM_CS: track 2.13 -> 17.0 mm, vias 0 -> 2
